Commit message: Adding SLAM toolset. Needs config.

File: description/robot_core.xacro (robot description, xacro)
@@ -21,4 +21,12 @@
     <!-- Base Link -->
     <link name="base_link">
+    </link>
+    <!-- Base Footprint Link -->
+    <joint name="base_footprint_joint" type="fixed">
+        <parent link="base_link"/>
+        <child link="base_footprint"/>
+        <origin xyz="0 0 0" rpy="0 0 0"/>
+    </joint>
+    <link name="base_footprint">
     </link>
     <!-- Chassis link -->
