Commit message: slam mapping added

File: description/lidar.xacro (robot description, xacro)
@@ -4,5 +4,5 @@
         <parent link="chassis"/>
         <child link="laser_frame"/>
-        <origin xyz="0.13565 0 0.09775" rpy="0 0 0"/>
+        <origin xyz="0.13565 0 0.09775" rpy="0 0 ${pi}"/>
     </joint>
     <link name="laser_frame">
